Commit message: added bioloid-halfarm urdf and launch file

File: bioloid_c_description/urdf/bioloid-halfarm.urdf (robot description, URDF)
Before this commit: robot loadscanner, 18 links, 17 joints
Links:
- removed link left_arm_link
- removed link right_arm_link
Joints:
- removed joint left_arm_joint
- removed joint right_arm_joint
- joint left_forearm_joint: origin xyz=0.0 0.0 -0.0675 rpy=0.0 0.0 0.0 -> xyz=0.0 0.023 -0.0145 rpy=0.0 0.0 0.0; parent left_arm_link -> left_shoulder_link
- joint right_forearm_joint: origin xyz=0.0 -0.0 -0.0675 rpy=0.0 0.0 0.0 -> xyz=0.0 -0.023 -0.0145 rpy=0.0 0.0 0.0; parent right_arm_link -> right_shoulder_link
